File: ELoad.kicad_sch (KiCad schematic)
At the start: 24 parts

Commit message: Schematic
Parts:
- removed U?: MCP41010, symbol Potentiometer_Digital:MCP41010
- added C?: 22uF, symbol Device:C_Small
- added J?: Conn_01x02, symbol Connector_Generic:Conn_01x02
- added Q?: Q_PMOS_GDS, symbol Device:Q_PMOS_GDS
- added Q?: Q_NPN_BEC, symbol Device:Q_NPN_BEC
- added R? (x5): 5R, symbol Device:R_Small
- added R?: 100kR, symbol Device:R_Small
- added R?: 650kR, symbol Device:R_Small
- added R?: 100R, symbol Device:R_Small
- added U?: MCP41010, symbol Potentiometer_Digital:MCP41010
Connections:
- net at Q?.1 (G): now also U?.1
- net at Q?.3 (S): now also U?.2 (-), R?.1, R?.1, R?.1, R?.1, R?.1
- net at SW?.1: now also Q?.1 (B), Q?.1 (B), R?.2
- net at SW?.2: now also C?.2, Q?.3 (C)
- net at U?.3 (+): now also U?.6 (PW0)
- net GND: now reaches Q?.2 (E)
- net GND: now also J?.2 (Pin_2), Q?.2 (E), R?.2, R?.2, R?.2, R?.2, R?.2, U?.4 (VSS), U?.7 (PB0)
- net at Q?.3 (C): now also Q?.1 (G), R?.2
- new net: J?.1 (Pin_1), Q?.3 (S), R?.1, R?.1
- new net: C?.1, R?.2
- new net +15V: Q?.2 (D), R?.1
- new net +3V3: U?.5 (PA0), U?.8 (VDD)
Other:
- moved on the sheet: C?, Q?, SW?, U?, U?A, U?B, U?C
